Commit message: update

File: rb_description/urdf/rb10_moveit.xacro (robot description, xacro)
@@ -1,5 +1,5 @@
 <?xml version="1.0"?>
 <!-- Cobot Robot -->
-<robot name="rb10" xmlns:xacro="http://www.ros.org/wiki/xacro">
+<robot name="RB10" xmlns:xacro="http://www.ros.org/wiki/xacro">
   <!-- Constants for robot dimensions -->
   <xacro:property name="PI" value="3.1415926535897931"/>

File: rb_moveit_config/config/rb10.ros2_control.xacro (robot description, xacro)
@@ -2,5 +2,5 @@
 <robot xmlns:xacro="http://www.ros.org/wiki/xacro">
     <xacro:macro name="rb10_ros2_control" params="name initial_positions_file">
-        <xacro:property name="initial_positions" value="${load_yaml(initial_positions_file)['initial_positions']}"/>
+        <xacro:property name="initial_positions" value="${xacro.load_yaml(initial_positions_file)['initial_positions']}"/>
         <ros2_control name="${name}" type="system">
             <hardware>

Commit message: attach Gripper

File: rb_description/urdf/rb10_moveit.xacro (robot description, xacro)
@@ -16,5 +16,5 @@
  <!--======================= Links =========================-->
  <!-- Base Footprint -->
- <link name="base_footprint">
+ <link name="base_link">
   <visual>
     <origin xyz="0 0 0" rpy="0 0 0"/>
@@ -138,16 +138,23 @@
 </link>
 <!-- TCP -->
-<link name="Tool_Center_Point">
-  <visual>
-     <origin xyz="${wrist2wrist} 0 ${-base2module1-pipe1_len-pipe2_len-wrist2wrist }" rpy="0 0 0"/>
-    <geometry>
-      <box size="0.001 0.001 0.001"/>
-    </geometry>
-    <material name="grey"/>
-  </visual>
+<link name="Tool_Vacuum">
+  <visual>
+    <origin xyz="0 -0.081 0" rpy="0 0 0"/>
+    <geometry>
+      <!-- <mesh filename="package://rb_description/meshes/visual/gripper_frame.stl" scale="0.001 0.001 0.001"/> -->
+      <box size="0.270 0.175 0.240"/>
+    </geometry>
+    <material name="grey"/>
+    <collision>
+      <box size="0.270 0.175 0.240"/>
+    </collision>
+  </visual>
+</link>
+<link name="tcp_link">
+  <origin xyz="0 0 0" rpy="0 0 0"/>
 </link>
 <!-- Joint -->
 <joint name="ground" type="fixed">
-  <parent link="base_footprint"/>
+  <parent link="base_link"/>
   <child link="Axis_0"/>
   <origin xyz="0 0 0" rpy="0 0 0"/>
@@ -193,7 +200,13 @@
 <joint name="Tool_Flange" type="fixed">
   <parent link="Axis_6"/>
-  <child link="Tool_Center_Point"/>
+  <child link="Tool_Vacuum"/>
   <origin xyz="0 ${-wrist2tcp} 0" rpy="0 0 0"/>
   <axis xyz="0 0 0"/>
 </joint>
+<joint name="tool_tcp" type="fixed">
+  <parent link="Tool_Vacuum"/>
+  <child link="tcp_link"/>
+  <origin xyz="0 0 0" rpy="0 0 0"/>
+  <axis xyz="0 0 0"/>
+</joint>
 </robot>
